File: PCB/N6480.kicad_pcb (KiCad board)
At the start: 2 copper layers, 44 parts

Commit message: PCB looks pretty much done. Just need copper fill and mounting holes.
Parts:
- removed the   at (147.0, 136.0)
- removed the   at (142.2, 135.2)
- added  : Resistor_SMD0805_HandSoldering_RevA_Date21Jun2010, Resistor_SMD0805_HandSoldering_RevA_Date21Jun2010, F.Cu at (180.0, 71.5)
- added  : Resistor_SMD0805_HandSoldering_RevA_Date21Jun2010, Resistor_SMD0805_HandSoldering_RevA_Date21Jun2010, F.Cu at (180.2, 84.0)
- added  : Resistor_SMD0805_HandSoldering_RevA_Date21Jun2010, Resistor_SMD0805_HandSoldering_RevA_Date21Jun2010, F.Cu at (135.8, 112.8)
- added 15/30KHz: Val**, PIN_ARRAY_2X1, F.Cu at (182.5, 75.5)
- added C104: V***, C1, F.Cu at (149.5, 28.2)
- added C1V5: C***, C1V5, F.Cu at (149.5, 17.8)
- added C1V5: C***, C1V5, F.Cu at (149.5, 23.8)
- added GND: Val**, SIL-1, F.Cu at (143.2, 33.2)
- added GND: Val**, PIN_ARRAY_1, F.Cu at (145.8, 131.0)
- added YUV/RGB: Val**, PIN_ARRAY_2X1, F.Cu at (182.5, 79.8)
- added c_0402: C***, c_0402, F.Cu at (163.2, 25.0)
- added c_0402: C***, c_0402, F.Cu at (162.5, 28.8)
- 220 uF: value Filter -> 3.3V Filter
- 220uF: renamed from C1.5V8V; value V*** -> 3.3V Filter
- 22uF: value Filter -> 1.2V Filter
- SOT223: value ASM1117-1.2 -> AZ1117CH-1.2
- moved VCC5 11.4 mm to (143.2, 31.0)
- renumbered 104 to C104
Routing:
- net (no net): track 3882.4 -> 4114.9 mm, vias 125 -> 133
Other:
- board outline added: 52.2 x 118.2 mm
- board text added: "N6480 - N64 to VGA Scaler"
- board text added: "https://github.com/Mikejmoffitt"

Commit message: PCB has copper fills. Beware: Every time kicad reopens it it'll break the copper ground links
Routing:
- net (no net): track 4114.9 -> 4448.1 mm
- added copper zone on B.Cu, net (none)
- added copper zone on F.Cu, net (none)

Commit message: Fixed mistake in logo and added holes
Parts:
- added 1PIN: P***, 1pin, F.Cu at (143.0, 18.0)
- added 1PIN: P***, 1pin, F.Cu at (138.0, 76.0)
- added 1PIN: P***, 1pin, F.Cu at (181.0, 128.0)
Changed lines of the file:
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@@
     (tracks 1683)
     (zones 0)
-    (modules 54)
+    (modules 57)
     (nets 1)
   )
   (page A3)
   (layers
-    (15 F.Cu signal hide)
+    (15 F.Cu signal)
     (0 B.Cu signal)
     (16 B.Adhes user hide)
-    (17 F.Adhes user)
+    (17 F.Adhes user hide)
     (18 B.Paste user hide)
     (19 F.Paste user)
@@
     (visible_elements FFFFFD3F)
     (pcbplotparams
-      (layerselection 3178497)
+      (layerselection 284196865)
       (usegerberextensions true)
       (excludeedgelayer true)
@@
       (outputformat 1)
       (mirror false)
-      (drillshape 1)
+      (drillshape 0)
       (scaleselection 1)
-      (outputdirectory ""))
+      (outputdirectory Out/))
   )
   (net 0 "")
@@
     )
   )
+  (module 1pin (layer F.Cu)
+    (at 143 18)
+    (descr "module 1 pin (ou trou mecanique de percage)")
+    (tags DEV)
+    (path 1pin)
+    (fp_text reference 1PIN (at 0 -3.048) (layer F.SilkS)
+      (effects (font (size 1.016 1.016) (thickness 0.254)))
+    )
+    (fp_text value P*** (at 0 2.794) (layer F.SilkS) hide
+      (effects (font (size 1.016 1.016) (thickness 0.254)))
+    )
+    (fp_circle (center 0 0) (end 0 -2.286) (layer F.SilkS) (width 0.381))
+    (pad 1 thru_hole circle (at 0 0) (size 4.064 4.064) (drill 3.048)
+      (layers *.Cu *.Mask F.SilkS)
+    )
+  )
+  (module 1pin (layer F.Cu)
+    (at 138 76)
+    (descr "module 1 pin (ou trou mecanique de percage)")
+    (tags DEV)
+    (path 1pin)
+    (fp_text reference 1PIN (at 0 -3.048) (layer F.SilkS)
+      (effects (font (size 1.016 1.016) (thickness 0.254)))
+    )
+    (fp_text value P*** (at 0 2.794) (layer F.SilkS) hide
+      (effects (font (size 1.016 1.016) (thickness 0.254)))
+    )
+    (fp_circle (center 0 0) (end 0 -2.286) (layer F.SilkS) (width 0.381))
+    (pad 1 thru_hole circle (at 0 0) (size 4.064 4.064) (drill 3.048)
+      (layers *.Cu *.Mask F.SilkS)
+    )
+  )
+  (module 1pin (layer F.Cu)
+    (at 181 128)
+    (descr "module 1 pin (ou trou mecanique de percage)")
+    (tags DEV)
+    (path 1pin)
+    (fp_text reference 1PIN (at 0 -3.048) (layer F.SilkS)
+      (effects (font (size 1.016 1.016) (thickness 0.254)))
+    )
+    (fp_text value P*** (at 0 2.794) (layer F.SilkS) hide
+      (effects (font (size 1.016 1.016) (thickness 0.254)))
+    )
+    (fp_circle (center 0 0) (end 0 -2.286) (layer F.SilkS) (width 0.381))
+    (pad 1 thru_hole circle (at 0 0) (size 4.064 4.064) (drill 3.048)
+      (layers *.Cu *.Mask F.SilkS)
+    )
+  )
   (gr_text "10K R" (at 180 74.75) (layer B.SilkS)
     (effects (font (size 0.5 0.5) (thickness 0.125)) (justify mirror))
@@
   (segment (start 158.77 103) (end 158 103) (width 0.8) (layer B.Cu) (net 0))
   (segment (start 158 103) (end 157 102) (width 0.8) (layer B.Cu) (net 0))
-  (segment (start 158.77 104.42) (end 160.42 104.42) (width 0.8) (layer B.Cu) (net 0) (status 400000))
+  (segment (start 158.77 104.42) (end 160.42 104.42) (width 0.8) (layer B.Cu) (net 0))
   (segment (start 160.42 104.42) (end 161 105) (width 0.8) (layer B.Cu) (net 0))
   (segment (start 143.58 102.67) (end 143.58 101.42) (width 0.8) (layer B.Cu) (net 0))
@@
   (segment (start 144 131) (end 145.75 129.25) (width 0.8) (layer B.Cu) (net 0))
   (segment (start 144 131) (end 144 129) (width 0.8) (layer B.Cu) (net 0))
-  (segment (start 153.655 127.25) (end 153.655 126.655) (width 0.8) (layer B.Cu) (net 0) (status C00000))
-  (segment (start 153.655 126.655) (end 152 125) (width 0.8) (layer B.Cu) (net 0) (status 400000))
+  (segment (start 153.655 127.25) (end 153.655 126.655) (width 0.8) (layer B.Cu) (net 0))
+  (segment (start 153.655 126.655) (end 152 125) (width 0.8) (layer B.Cu) (net 0))
   (segment (start 152.25 127.25) (end 152.25 128.75) (width 0.8) (layer B.Cu) (net 0))
   (segment (start 153.655 127.25) (end 152.25 127.25) (width 0.8) (layer B.Cu) (net 0))
@@
   (segment (start 184 78) (end 185 78) (width 0.8) (layer B.Cu) (net 0))
   (segment (start 185 74) (end 185 78) (width 0.8) (layer B.Cu) (net 0))
-  (segment (start 183.77 75.5) (end 183.77 75.23) (width 0.8) (layer B.Cu) (net 0) (status C00000))
-  (segment (start 183.77 75.23) (end 185 74) (width 0.8) (layer B.Cu) (net 0) (status 400000))
-  (segment (start 183.77 78) (end 183.77 75.5) (width 0.8) (layer B.Cu) (net 0) (status 800000))
+  (segment (start 183.77 75.5) (end 183.77 75.23) (width 0.8) (layer B.Cu) (net 0))
+  (segment (start 183.77 75.23) (end 185 74) (width 0.8) (layer B.Cu) (net 0))
+  (segment (start 183.77 78) (end 183.77 75.5) (width 0.8) (layer B.Cu) (net 0))
   (segment (start 162.25 76.75) (end 162.25 77.25) (width 0.8) (layer B.Cu) (net 0))
   (segment (start 162.25 77.25) (end 163 78) (width 0.8) (layer B.Cu) (net 0))
@@
   (segment (start 162.25 76.75) (end 161 78) (width 0.8) (layer B.Cu) (net 0))
   (segment (start 174.5 47) (end 172 47) (width 0.8) (layer B.Cu) (net 0))
-  (segment (start 168 47.52) (end 168 52) (width 0.8) (layer B.Cu) (net 0) (status 400000))
+  (segment (start 168 47.52) (end 168 52) (width 0.8) (layer B.Cu) (net 0))
   (segment (start 168 52) (end 167 53) (width 0.8) (layer B.Cu) (net 0))
-  (segment (start 174.5 51.7468) (end 174.5 51.5) (width 0.8) (layer B.Cu) (net 0) (status C00000))
-  (segment (start 174.5 51.5) (end 178 48) (width 0.8) (layer B.Cu) (net 0) (status 400000))
-  (segment (start 174.5 51.5) (end 171 48) (width 0.8) (layer B.Cu) (net 0) (status 400000))
-  (segment (start 174.5 55) (end 174.5 60.655) (width 0.8) (layer B.Cu) (net 0) (status 800000))
-  (segment (start 174.5 60.655) (end 174.405 60.75) (width 0.8) (layer B.Cu) (net 0) (status C00000))
+  (segment (start 174.5 51.7468) (end 174.5 51.5) (width 0.8) (layer B.Cu) (net 0))
+  (segment (start 174.5 51.5) (end 178 48) (width 0.8) (layer B.Cu) (net 0))
+  (segment (start 174.5 51.5) (end 171 48) (width 0.8) (layer B.Cu) (net 0))
+  (segment (start 174.5 55) (end 174.5 60.655) (width 0.8) (layer B.Cu) (net 0))
+  (segment (start 174.5 60.655) (end 174.405 60.75) (width 0.8) (layer B.Cu) (net 0))
   (segment (start 174.5 55) (end 177 55) (width 0.8) (layer B.Cu) (net 0))
   (segment (start 174.5 55) (end 173 55) (width 0.8) (layer B.Cu) (net 0))
@@
   (segment (start 151 16.02) (end 152.98 16.02) (width 0.8) (layer B.Cu) (net 0))
   (segment (start 152.98 16.02) (end 153 16) (width 0.8) (layer B.Cu) (net 0))
-  (segment (start 150.77 17.75) (end 152.25 17.75) (width 0.8) (layer B.Cu) (net 0) (status 400000))
+  (segment (start 150.77 17.75) (end 152.25 17.75) (width 0.8) (layer B.Cu) (net 0))
   (segment (start 152.25 17.75) (end 153 17) (width 0.8) (layer B.Cu) (net 0))
   (segment (start 162.667 119.845) (end 161.595 119.845) (width 0.8) (layer F.Cu) (net 0))
@@
     (polygon
       (pts
-        (xy 141 55) (xy 136 55) (xy 136 54) (xy 141 54)
+        (xy 141 55) (xy 136 55) (xy 136 54) (xy 138 54) (xy 138 53)
+        (xy 139 53) (xy 139 54) (xy 141 54) (xy 141 55)
+      )
+    )
+  )
+  (zone (net 0) (net_name "") (layer F.SilkS) (hatch none 0.508)
+    (connect_pads (clearance 0.508))
+    (min_thickness 0.254)
+    (fill (arc_segments 16) (thermal_gap 0.508) (thermal_bridge_width 0.508))
+    (polygon
+      (pts
+        (xy 141 52) (xy 140 52) (xy 140 53) (xy 139 53) (xy 139 52)
+        (xy 136 52) (xy 136 51) (xy 141 51)
       )
     )

Commit message: Few more changes
Routing:
- net (no net): track 4448.1 -> 4472.8 mm, vias 133 -> 134
Changed lines of the file:
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@@
     (thickness 1.6)
     (drawings 46)
-    (tracks 1683)
+    (tracks 1712)
     (zones 0)
     (modules 57)
@@
   (layers
     (15 F.Cu signal)
-    (0 B.Cu signal)
+    (0 B.Cu signal hide)
     (16 B.Adhes user hide)
     (17 F.Adhes user hide)
@@
     (effects (font (size 0.75 0.75) (thickness 0.1875)))
   )
+  (segment (start 183.75 82) (end 183.75 79.77) (width 0.8) (layer F.Cu) (net 0) (status 800000))
+  (segment (start 183.77 77.48) (end 183.77 75.5) (width 0.8) (layer F.Cu) (net 0) (status 800000))
+  (segment (start 183.75 77.5) (end 183.77 77.48) (width 0.8) (layer F.Cu) (net 0))
+  (segment (start 183.75 79.77) (end 183.75 77.5) (width 0.8) (layer F.Cu) (net 0) (status 400000))
+  (segment (start 183.77 81.48) (end 183.77 82.73) (width 0.8) (layer B.Cu) (net 0))
+  (segment (start 183.77 82.73) (end 183.75 82.75) (width 0.8) (layer B.Cu) (net 0))
+  (segment (start 185.25 78) (end 185.25 81) (width 0.8) (layer B.Cu) (net 0))
+  (segment (start 167.25 95.75) (end 168 95.75) (width 0.8) (layer B.Cu) (net 0))
+  (segment (start 167.25 95.75) (end 167.25 97.25) (width 0.8) (layer B.Cu) (net 0))
+  (segment (start 167.25 111) (end 166.75 111) (width 0.8) (layer B.Cu) (net 0))
+  (segment (start 166.75 111) (end 165.75 112) (width 0.8) (layer B.Cu) (net 0))
+  (segment (start 167.25 114) (end 168.5 114) (width 0.8) (layer B.Cu) (net 0))
+  (segment (start 167.25 123.75) (end 167.75 123.75) (width 0.8) (layer B.Cu) (net 0))
+  (segment (start 167.75 123.75) (end 168.25 124.25) (width 0.8) (layer B.Cu) (net 0))
+  (segment (start 167.25 121.75) (end 166.25 121.75) (width 0.8) (layer B.Cu) (net 0))
+  (segment (start 167.25 119.25) (end 168.25 119.25) (width 0.8) (layer B.Cu) (net 0))
+  (segment (start 167.25 116.75) (end 166 116.75) (width 0.8) (layer B.Cu) (net 0))
+  (segment (start 167.125 124.375) (end 166.125 124.375) (width 0.8) (layer B.Cu) (net 0))
+  (segment (start 166.125 124.375) (end 165.75 124) (width 0.8) (layer B.Cu) (net 0))
+  (segment (start 165.5 109.25) (end 167.5 109.25) (width 0.8) (layer B.Cu) (net 0))
+  (via (at 135.75 111.5) (size 0.889) (layers F.Cu B.Cu) (net 0))
+  (segment (start 138.73 112.83) (end 137.08 112.83) (width 0.254) (layer B.Cu) (net 0))
+  (segment (start 137.08 112.83) (end 135.75 111.5) (width 0.254) (layer B.Cu) (net 0))
+  (segment (start 135.75 111.5) (end 135.75 111.44952) (width 0.8) (layer F.Cu) (net 0))
   (segment (start 158.77 103) (end 158 103) (width 0.8) (layer B.Cu) (net 0))
   (segment (start 158 103) (end 157 102) (width 0.8) (layer B.Cu) (net 0))
@@
   (segment (start 184 78) (end 182 78) (width 0.8) (layer B.Cu) (net 0))
   (segment (start 183.77 78) (end 184 78) (width 0.8) (layer B.Cu) (net 0))
-  (segment (start 184 78) (end 185 78) (width 0.8) (layer B.Cu) (net 0))
+  (segment (start 184 78) (end 185.25 78) (width 0.8) (layer B.Cu) (net 0))
+  (segment (start 185.25 78) (end 185 78) (width 0.8) (layer B.Cu) (net 0))
   (segment (start 185 74) (end 185 78) (width 0.8) (layer B.Cu) (net 0))
   (segment (start 183.77 75.5) (end 183.77 75.23) (width 0.8) (layer B.Cu) (net 0))
@@
   (segment (start 135.75 116.25) (end 136.98 117.48) (width 0.254) (layer F.Cu) (net 0))
   (segment (start 136.98 117.48) (end 136.98 119.25) (width 0.254) (layer F.Cu) (net 0))
-  (segment (start 138.73 112.83) (end 137.08 112.83) (width 0.254) (layer B.Cu) (net 0))
-  (segment (start 137.08 112.83) (end 135.75 111.5) (width 0.254) (layer B.Cu) (net 0))
   (segment (start 141.05048 116) (end 143.912 116) (width 0.254) (layer F.Cu) (net 0))
   (segment (start 143.912 116) (end 144.714 115.198) (width 0.254) (layer F.Cu) (net 0))
@@
   (segment (start 165.5 109.25) (end 167.25 111) (width 0.8) (layer B.Cu) (net 0))
   (segment (start 163.5 128) (end 160.77 128) (width 0.8) (layer B.Cu) (net 0))
-  (segment (start 167.25 124.25) (end 163.5 128) (width 0.8) (layer B.Cu) (net 0))
-  (segment (start 167.25 111) (end 167.25 124.25) (width 0.8) (layer B.Cu) (net 0))
+  (segment (start 167.25 124.25) (end 167.125 124.375) (width 0.8) (layer B.Cu) (net 0))
+  (segment (start 167.125 124.375) (end 163.5 128) (width 0.8) (layer B.Cu) (net 0))
+  (segment (start 167.25 111) (end 167.25 114) (width 0.8) (layer B.Cu) (net 0))
+  (segment (start 167.25 114) (end 167.25 116.75) (width 0.8) (layer B.Cu) (net 0))
+  (segment (start 167.25 116.75) (end 167.25 119.25) (width 0.8) (layer B.Cu) (net 0))
+  (segment (start 167.25 119.25) (end 167.25 121.75) (width 0.8) (layer B.Cu) (net 0))
+  (segment (start 167.25 121.75) (end 167.25 123.75) (width 0.8) (layer B.Cu) (net 0))
+  (segment (start 167.25 123.75) (end 167.25 124.25) (width 0.8) (layer B.Cu) (net 0))
   (segment (start 160.77 128) (end 160.77 128.73) (width 0.8) (layer F.Cu) (net 0))
   (segment (start 160.77 128.73) (end 159.5 130) (width 0.8) (layer F.Cu) (net 0))
